File: Hardware_Design/Mind_Speak/Mind_Speak.kicad_sch (KiCad schematic)
At the start: 43 parts, among them J1 microSD, P1 S2B-PH-SM4-TB_LF__SN_, U1 CDBU0130L, U2 LP5907MFX-3.3, U3 TCM828ECT713, U4 TLV70025_SOT23-5, U5 TPS72325DBV, U6 LIS3DH, U7 SN74LVC1G32DCKR, U8 ADS1299

Commit message: Edited The Schema
Parts:
- removed C3, C4: 10uF, PCM_SparkFun-Capacitor:C_0603_1608Metric, symbol PCM_SparkFun-Capacitor:10uF_0603_10V_20%
- removed U3: TCM828ECT713, Package_TO_SOT_SMD:SOT-23-5, symbol TCM828ECT713:TCM828ECT713
- added C33, C34, C35: 1.0uF, PCM_SparkFun-Capacitor:C_0402_1005Metric, symbol PCM_SparkFun-Capacitor:1.0uF_0402_16V_10%
- added C36, C37, C38, C39, C4: CKCL44X7R1H102M085AA, TDK_Library:CKCL44_TDK, symbol CKCL44X7R1H102M085AA:CKCL44X7R1H102M085AA
- added D1, D2, D3, D4, D5: TPD4E1B06DCKR, TI_Library:TVS_TPD4E1B06DCKR, symbol TPD4E1B06DCKR:TPD4E1B06DCKR
- added J4: Conn_01x08_Pin, Connector_PinHeader_2.54mm:PinHeader_1x08_P2.54mm_Vertical, symbol Connector:Conn_01x08_Pin
- added J5: Conn_01x02_Pin, Connector_PinHeader_2.54mm:PinHeader_1x02_P2.54mm_Vertical, symbol Connector:Conn_01x02_Pin
- added J6, J7: Conn_01x04_Pin, Connector_PinHeader_2.54mm:PinHeader_1x04_P2.54mm_Vertical, symbol Connector:Conn_01x04_Pin
- added J8: Conn_02x13_Odd_Even, Connector_PinHeader_2.54mm:PinHeader_2x13_P2.54mm_Horizontal, symbol Connector_Generic:Conn_02x13_Odd_Even
- added RN1, RN2, RN3, RN4, RN5: CAY16-2201F4LF, Bourns_Library:RESCAF80P320X160X60-8N, symbol Bourns_Library:CAY16-2201F4LF
- added U10: PIC32MX250F128B-I_SS, MicroChip_Library:SOP65P780X200-28N, symbol PIC32MX250F128B-I_SS:PIC32MX250F128B-I_SS
- added U3: NINA-B30x, U_Blox_Library:XCVR_NINA-B306-00B, symbol NINA-B306-00B:NINA-B30x
- added U9: TPS60403DBV, Package_TO_SOT_SMD:SOT-23-5, symbol Regulator_SwitchedCapacitor:TPS60403DBV
- U1: footprint CDBU -> (none)
Connections:
- net +3V3: now also C33.1, U9.2 (IN)
- net -V: now also C35.1, U9.1 (OUT)
- net GNDA: now also C33.2, C35.2, U9.4 (GND)
- new net: C34.2, U9.3 (C_{FLY-})
- new net: C34.1, U9.5 (C_{FLY+})
- new net EAGP: U3.EAGP1 (EAGP), U3.EAGP2 (EAGP), U3.EAGP3 (EAGP), U3.EAGP4 (EAGP)
- new net EGP: U3.EGP1 (EGP), U3.EGP10 (EGP), U3.EGP11 (EGP), U3.EGP12 (EGP), U3.EGP2 (EGP), U3.EGP3 (EGP), U3.EGP4 (EGP), U3.EGP5 (EGP), U3.EGP6 (EGP), U3.EGP7 (EGP), U3.EGP8 (EGP), U3.EGP9 (EGP)
- new net GND: U3.12 (GND), U3.14 (GND), U3.26 (GND), U3.30 (GND), U3.53 (GND), U3.6 (GND)
- new net VSS: U10.19 (VSS), U10.8 (VSS)
Other:
- note added: "ADS_DECOUBLING"
- note added: "Imax = 80mA Vmax = 0.3V Pmax = 0.024W"
- note added: "OR_GATE"
- note removed: "Imax = 50mA Vmax = 6V Pmax = 300mW"
- note removed: "Should Be Changed"
- moved on the sheet: C12, C13, C14, C15, C16, C17, C18, C19, C23, C24, C25, C26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

Commit message: Edit in The Schematic
Parts:
- removed RN1: CAY16-2201F4LF, Bourns_Library:RESCAF80P320X160X60-8N, symbol Bourns_Library:CAY16-2201F4LF
- added D6: TPD4E1B06DCKR, TI_Library:TVS_TPD4E1B06DCKR, symbol TPD4E1B06DCKR:TPD4E1B06DCKR
- added RN6: CAY16-2201F4LF, Bourns_Library:RESCAF80P320X160X60-8N, symbol Bourns_Library:CAY16-2201F4LF
Connections:
- net +2.5VA: now also D6.2 (IO2)
- net BIAS_DRV: now also C39.1, RN6.8
- net GNDA: now also C36.5, C36.6, C36.7, C36.8, C37.5, C37.6, C37.7, C37.8, C38.5, C38.6, C38.7, C38.8, C39.2, C39.5, C39.6, C39.7, C39.8, C4.5, C4.6, C4.7, C4.8, D1.3 (GND), D2.3 (GND), D3.3 (GND), D4.3 (GND), D5.3 (GND), D6.1 (IO1), D6.3 (GND), RN6.2, RN6.7
- net IN1_N: now also C4.1, RN2.8
- net IN1_P: now also C4.2, RN2.7
- net IN2_N: now also C36.3, RN3.6
- net IN2_P: now also C36.4, RN3.5
- net IN3_N: now also C36.1, RN3.8
- net IN3_P: now also C36.2, RN3.7
- net IN4_N: now also C37.3, RN4.6
- net IN4_P: now also C37.4, RN4.5
- net IN5_N: now also C37.1, RN4.8
- net IN5_P: now also C37.2, RN4.7
- net IN6_N: now also C38.3, RN5.6
- net IN6_P: now also C38.4, RN5.5
- net IN7_N: now also C38.1, RN5.8
- net IN7_P: now also C38.2, RN5.7
- net IN8_N: now also C39.3, RN6.6
- net IN8_P: now also C39.4, RN6.5
- net VSSA: now also D1.4 (IO3)
- net _SRB1: now also C4.4, RN2.5
- net _SRB2: now also C4.3, RN2.6
- net 8N: now reaches D5.2 (IO2)
- net 8N: now also RN6.3
- net 7N: now reaches D5.4 (IO3)
- net 7N: now also RN5.1
- net 8P: now reaches D5.5 (IO4)
- net 8P: now also RN6.4
- net 7P: now reaches RN5.2
- net 7P: now also D4.1 (IO1)
- net 6N: now reaches RN5.3
- net 6N: now also D4.2 (IO2)
- net 6P: now reaches RN5.4
- net 6P: now also D4.5 (IO4)
- net 5N: now reaches RN4.1
- net 5N: now also D4.4 (IO3)
- net 5P: now reaches RN4.2
- net 5P: now also D3.1 (IO1)
- net 4N: now reaches RN4.3
- net 4N: now also D3.2 (IO2)
- net 4P: now reaches RN4.4
- net 4P: now also D3.5 (IO4)
- net 1P: now reaches D1.1 (IO1)
- net 1P: now also RN2.2
- net SRB2: now reaches D1.2 (IO2)
- net SRB2: now also RN2.3
- net SRB1: now reaches D1.5 (IO4)
- net SRB1: now also RN2.4
- net 3N: now reaches D3.4 (IO3)
- net 3N: now also RN3.1
- net 3P: now reaches D2.1 (IO1)
- net 3P: now also RN3.2
- net 2N: now reaches D2.2 (IO2)
- net 2N: now also RN3.3
- net 1N: now reaches D2.4 (IO3)
- net 1N: now also RN2.1
- net 2P: now reaches D2.5 (IO4)
- net 2P: now also RN3.4
- new net BIAS: D6.4 (IO3), RN6.1
- no-connect marks 12 -> 20
Other:
- moved on the sheet: C10, C11, C12, C13, C14, C15, C16, C17, C18, C19, C20, C21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
