File: Hardware_Design/Mind_Speak_(Dongle_Board)/Mind_Speak_(Dongle_Board).kicad_sch (KiCad schematic)
At the start: 3 parts, among them J1 USB_A, SW1 SPDT_Slide_SMD_6.7x2.6mm, U1 FT231XQ

Commit message: Edit In Dongle Board
Parts:
- added C1: 10nF, PCM_SparkFun-Capacitor:C_0402_1005Metric, symbol PCM_SparkFun-Capacitor:10nF_0402_25V_10%
- added C2, C3: 47pF, Capacitors SMD:CAPC0603X33N, symbol PCM_SparkFun-Capacitor:47pF_0603_50V_5%
- added D1: PESD5V0S1UL, Diode_SMD:D_SOD-882, symbol Diode:PESD5V0S1UL
- added D2, D3: CG0402MLC-05LG, ESD_SMD:CG0402MLC-05LG, symbol Device:CG0402MLC-05LG
- added D4: Green, PCM_SparkFun-LED:LED_0603_1608Metric_Green, symbol PCM_SparkFun-LED:LED_Green_0603
- added D5: Red, PCM_SparkFun-LED:LED_0603_1608Metric_Red, symbol PCM_SparkFun-LED:LED_Red_0603
- added F1: 0.5A, PCM_SparkFun-Fuse:1812, symbol PCM_SparkFun-Fuse:Fuse 16V/2.5A/5.0A
- added J2: Conn_01x07_Pin, Connector_PinHeader_2.54mm:PinHeader_1x07_P2.54mm_Vertical, symbol Connector:Conn_01x07_Pin
- added J3: Conn_01x05_Pin, Connector_PinHeader_2.54mm:PinHeader_1x05_P2.54mm_Vertical, symbol Connector:Conn_01x05_Pin
- added L1, L2: 30 Ohm, PCM_SparkFun-Capacitor:C_0402_1005Metric, symbol PCM_SparkFun-Coil:Ferrite_120Ohm_0402_0.3A
- added R1, R2: 22, PCM_SparkFun-Resistor:R_0402_1005Metric, symbol PCM_SparkFun-Resistor:22_0402
- added R3: 10k, PCM_SparkFun-Resistor:R_0402_1005Metric, symbol PCM_SparkFun-Resistor:10k_0402
- added R4, R5: 330, PCM_SparkFun-Resistor:R_0402_1005Metric, symbol PCM_SparkFun-Resistor:330_0402
- added R6, R7: 1k, PCM_SparkFun-Resistor:R_0402_1005Metric, symbol PCM_SparkFun-Resistor:1k_0402
- J1: footprint (none) -> Connector_USB:MOLEX_48037-1000
Connections:
- net at J1.1 (VBUS): now also C1.1, L2.1
- net at J1.2 (D-): now also C3.1, D3.2, R2.1
- net at J1.3 (D+): now also C2.1, D2.2, R1.1
- net at J1.4 (GND): now also C1.2, L1.2
- net at U1.1 (RXD): now also R7.1
- net 3.3V: now reaches U1.10 (3V3OUT)
- net 3.3V: now also U1.11 (~{RESET}), U1.20 (VCCIO), D4.2 (A), D5.2 (A), R3.2
- net VBUS: now reaches U1.12 (VCC)
- net VBUS: now also D1.1 (K), F1.2
- net GND: now reaches U1.13 (GND)
- net GND: now also U1.21 (GND), U1.3 (GND), C2.2, C3.2, D1.2 (A), D2.1, D3.1, L1.1
- net at U1.14 (CBUS1): now also R5.1
- net at U1.17 (TXD): now also R6.1
- net DTR: now reaches U1.18 (~{DTR})
- net DTR: now also SW1.2
- net at U1.7 (CBUS2): now also R4.1
- net USB_D+: now reaches U1.8 (USBDP)
- net USB_D+: now also R1.2
- net USB_D-: now reaches U1.9 (USBDM)
- net USB_D-: now also R2.2
- net RFD_RESET: now reaches SW1.1 (A)
- net GPIO6: now reaches SW1.3 (C)
- net GPIO6: now also R3.1
- new net: D5.1 (K), R4.2
- new net: F1.1, L2.2
- new net: D4.1 (K), R5.2
- new net FTDI_RX: R7.2
- new net FTDI_TX: R6.2
- no-connect marks 1 -> 8
Other:
- moved on the sheet: J1, SW1, U1

Commit message: Edit The main Board
Parts:
- added U2: NINA-B30x, U_Blox_Library:XCVR_NINA-B306-00B, symbol NINA-B306-00B:NINA-B30x
Connections:
- net GND: now also U2.12 (GND), U2.14 (GND), U2.26 (GND), U2.30 (GND), U2.53 (GND), U2.6 (GND)
- new net EAGP: U2.EAGP1 (EAGP), U2.EAGP2 (EAGP), U2.EAGP3 (EAGP), U2.EAGP4 (EAGP)
- new net EGP: U2.EGP1 (EGP), U2.EGP10 (EGP), U2.EGP11 (EGP), U2.EGP12 (EGP), U2.EGP2 (EGP), U2.EGP3 (EGP), U2.EGP4 (EGP), U2.EGP5 (EGP), U2.EGP6 (EGP), U2.EGP7 (EGP), U2.EGP8 (EGP), U2.EGP9 (EGP)
Other:
- moved on the sheet: C1, C2, C3, D1, D2, D3, D4, D5, F1, J1, J2, J3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

Commit message: Last Edit in main and dongle boards
Parts:
- removed J2: Conn_01x07_Pin, Connector_PinHeader_2.54mm:PinHeader_1x07_P2.54mm_Vertical, symbol Connector:Conn_01x07_Pin
- removed R3: 10k, PCM_SparkFun-Resistor:R_0402_1005Metric, symbol PCM_SparkFun-Resistor:10k_0402
- removed SW1: SPDT_Slide_SMD_6.7x2.6mm, Button_Switch_SMD:SW_SPDT_Shouhan_MSK12C02, symbol PCM_SparkFun-Switch:SPDT_Slide_SMD_6.7x2.6mm
- added C11: 10uF, PCM_SparkFun-Capacitor:C_0603_1608Metric, symbol PCM_SparkFun-Capacitor:10uF_0603_10V_20%
- added C13: 0.1uF, PCM_SparkFun-Capacitor:C_0402_1005Metric, symbol PCM_SparkFun-Capacitor:0.1uF_0402_16V_10%
- added J4: Conn_01x05_Pin, Connector_PinHeader_2.54mm:PinHeader_1x05_P2.54mm_Vertical, symbol Connector:Conn_01x05_Pin
- added SW3: SW_MEC_5E, Button_Switch_SMD:SW_Push_1P1T_NO_Vertical_Wuerth_434133025816, symbol Switch:SW_MEC_5E
- added SW4: SPDT_Slide_SMD_6.7x2.6mm, Button_Switch_SMD:SW_SPDT_Shouhan_MSK12C02, symbol PCM_SparkFun-Switch:SPDT_Slide_SMD_6.7x2.6mm
Connections:
- net EGP is gone; now on net EAGP: U2.EGP1 (EGP), U2.EGP10 (EGP), U2.EGP11 (EGP), U2.EGP12 (EGP), U2.EGP2 (EGP), U2.EGP3 (EGP), U2.EGP4 (EGP), U2.EGP5 (EGP), U2.EGP6 (EGP), U2.EGP7 (EGP), U2.EGP8 (EGP), U2.EGP9 (EGP)
- net GND is gone; now on net EAGP: C2.2, C3.2, D1.2 (A), D2.1, D3.1, L1.1, U1.13 (GND), U1.21 (GND), U1.3 (GND), U2.12 (GND), U2.14 (GND), U2.26 (GND), U2.30 (GND), U2.53 (GND), U2.6 (GND)
- net 3.3V: now also C13.1
- net EAGP: now also J3.5 (Pin_5), C11.2, C13.2, SW3.1, SW3.2
- net FTDI_RX: now also U2.2 (GPIO_2)
- net FTDI_TX: now also U2.3 (GPIO_3)
- net NINA_VCC: now reaches J3.1 (Pin_1)
- net NINA_VCC: now also SW4.3 (C)
- net SWD_CLK: now reaches J3.2 (Pin_2)
- net SWD_CLK: now also U2.11 (SWDCLK)
- net SWD_IO: now reaches J3.3 (Pin_3)
- net SWD_IO: now also U2.15 (SWDIO)
- net NINA_RST: now reaches J3.4 (Pin_4)
- net NINA_RST: now also U2.19 (~{RESET}), SW3.3 (K), SW3.4 (A)
- net NINA_PWR: now reaches U2.10 (VCC)
- net NINA_PWR: now also U2.9 (VCC_IO), C11.1, SW4.2
- net at U2.35 (GPIO_35): now also J4.5 (Pin_5)
- net at U2.36 (GPIO_36): now also J4.4 (Pin_4)
- net at U2.37 (GPIO_37): now also J4.3 (Pin_3)
- net at U2.38 (GPIO_38): now also J4.2 (Pin_2)
- net at U2.39 (GPIO_39): now also J4.1 (Pin_1)
- net DTR: no longer names the net of U1.18 (~{DTR})
- new net +3V3: SW4.1 (A)
- no-connect marks 8 -> 46
Other:
- note added: "BLE_INTERFACING"
- note added: "NINA_RX"
- note added: "NINA_TX"
- moved on the sheet: J3, U2

Commit message: Edit in Dongle Layout
Parts:
- removed SW4: SPDT_Slide_SMD_6.7x2.6mm, Button_Switch_SMD:SW_SPDT_Shouhan_MSK12C02, symbol PCM_SparkFun-Switch:SPDT_Slide_SMD_6.7x2.6mm
- added S1: SSSS811101, ALPS_Library:SW_SSSS811101, symbol SSSS811101:SSSS811101
- C1, C13: LINK (none) -> https://eu.mouser.com/en/ProductDetail/YAGEO/CC0402KRX7R7BB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; VENDOR (none) -> Mouser
- C11: LINK (none) -> https://www.lcsc.com/product-detail/C710916.html?s_z=n_q_GR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; VENDOR (none) -> LCSC
- C2, C3: footprint Capacitors SMD:CAPC0603X33N -> PCM_SparkFun-Capacitor:C_0402_1005Metric; LINK (none) -> https://eu.mouser.com/en/ProductDetail/Murata-Electronics/G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; VENDOR (none) -> Mouser
- D1: value PESD5V0S1UL -> ESDALC6V1-1M2; LINK (none) -> https://www.lcsc.com/product-detail/C2649894.html?s_z=n_q_E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; VENDOR (none) -> LCSC
- D2, D3: LINK (none) -> https://eu.mouser.com/en/ProductDetail/Bourns/CG0402MLC-05L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; VENDOR (none) -> Mouser
- D4: LINK (none) -> https://eu.mouser.com/en/ProductDetail/LITEON/LTST-C191KGKT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; VENDOR (none) -> Mouser
- D5: LINK (none) -> https://eu.mouser.com/en/ProductDetail/LITEON/LTST-C191KRKT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; VENDOR (none) -> Mouser
- F1: LINK (none) -> https://eu.mouser.com/en/ProductDetail/Bourns/MF-MSMF050-2?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; VENDOR (none) -> Mouser
- J1: LINK (none) -> https://eu.mouser.com/en/ProductDetail/Molex/48037-1000?qs=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; VENDOR (none) -> Mouser
- J3, J4: LINK (none) -> https://microohm-eg.com/pin-header-2-54mm-1x40-pin-male-sin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; VENDOR (none) -> MicroOhm
- L1, L2: LINK (none) -> https://www.lcsc.com/product-detail/C275480.html?s_z=n_q_MP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; VENDOR (none) -> LCSC
- R1, R2: LINK (none) -> https://eu.mouser.com/en/ProductDetail/YAGEO/RC0402FR-0722R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; VENDOR (none) -> Mouser
- R4, R5: LINK (none) -> https://eu.mouser.com/en/ProductDetail/YAGEO/RC0402JR-07330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; VENDOR (none) -> Mouser
- R6, R7: LINK (none) -> https://eu.mouser.com/en/ProductDetail/YAGEO/RT0402FRE071KL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; VENDOR (none) -> Mouser
- SW3: LINK (none) -> https://eu.mouser.com/en/ProductDetail/CK/PTS810SJK250SMTR-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; VENDOR (none) -> Mouser
- U1: LINK (none) -> https://www.lcsc.com/product-detail/C132159.html?s_z=n_q_FT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; VENDOR (none) -> LCSC
- U2: LINK (none) -> https://www2.mouser.com/en/ProductDetail/u-blox/NINA-B306-0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; VENDOR (none) -> Mouser
Connections:
- net 3.3V is gone; now on net +3V3: C13.1, D4.2 (A), D5.2 (A), U1.10 (3V3OUT), U1.11 (~{RESET}), U1.20 (VCCIO)
- net +3V3: now also S1.1
- net NINA_PWR: now also S1.2
- net NINA_VCC: now also S1.3

Commit message: Dongle Layout Finished
Parts:
- added C14: 0.1uF, PCM_SparkFun-Capacitor:C_0402_1005Metric, symbol PCM_SparkFun-Capacitor:0.1uF_0402_16V_10%
Connections:
- net EAGP: now also C14.2
- net NINA_PWR: now also C14.1
- net SWD_CLK: now also J3.3 (Pin_3); no longer J3.2 (Pin_2)
- net SWD_IO: now also J3.2 (Pin_2); no longer J3.3 (Pin_3)
- net at J4.1 (Pin_1): now also U2.23 (GPIO_23); no longer U2.39 (GPIO_39)
- net at J4.2 (Pin_2): now also U2.22 (GPIO_22); no longer U2.38 (GPIO_38)
- net at J4.3 (Pin_3): now also U2.21 (GPIO_21); no longer U2.37 (GPIO_37)
- net at J4.4 (Pin_4): now also U2.20 (GPIO_20); no longer U2.36 (GPIO_36)
- net at J4.5 (Pin_5): now also U2.18 (GPIO_18); no longer U2.35 (GPIO_35)
Other:
- note added: "FT231XQ"
- note added: "NINA_B306-01B"
- note added: "NINA_POWER_SWITCHING"
- note added: "Note: You can power nina from USB source or External 3.3V Source like (SWD_VCC) NINA_VCC -> Ex. (SWD_VCC) +3V3 -> USB Source"
- note added: "USB"
- moved on the sheet: C11, J3, J4, S1, SW3, U2

Commit message: Edit In Layout Of Main Board
Connections:
- net EAGP: now also J1.SH (Shield), S1.4 (SHIELD)
- no-connect marks 46 -> 45
Changed lines of the file:
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@@
 	)
 	(no_connect
-		(at 20.32 53.34)
-	)
-	(no_connect
 		(at 134.62 135.89)
 	)
@@
 	(wire
 		(pts
+			(xy 20.32 57.15) (xy 20.32 53.34)
+		)
+		(stroke
+			(width 0)
+			(type default)
+		)
+	)
+	(wire
+		(pts
 			(xy 219.71 80.01) (xy 222.25 80.01)
 		)
@@
 		)
 		(stroke
-			(width 0)
-			(type default)
+			(width 0.5)
+			(type solid)
 		)
 	)
@@
 		)
 		(stroke
-			(width 0)
-			(type default)
+			(width 0.5)
+			(type solid)
 		)
 	)
@@
 		)
 		(stroke
-			(width 0)
-			(type default)
+			(width 0.5)
+			(type solid)
 		)
 	)
@@
 		)
 		(stroke
-			(width 0)
-			(type default)
+			(width 0.5)
+			(type solid)
 		)
 	)
@@
 		)
 		(stroke
-			(width 0)
-			(type default)
+			(width 0.5)
+			(type solid)
 		)
 	)
@@
 	(wire
 		(pts
+			(xy 209.55 125.73) (xy 213.36 125.73)
+		)
+		(stroke
+			(width 0)
+			(type default)
+		)
+	)
+	(wire
+		(pts
 			(xy 40.64 31.75) (xy 40.64 30.48)
 		)
@@
 		)
 		(stroke
-			(width 0)
-			(type default)
+			(width 0.5)
+			(type solid)
 		)
 	)
@@
 		)
 		(stroke
-			(width 0)
-			(type default)
+			(width 0.5)
+			(type solid)
 		)
 	)
@@
 		)
 		(stroke
-			(width 0)
-			(type default)
+			(width 0.5)
+			(type solid)
 		)
 	)
@@
 		)
 		(stroke
-			(width 0)
-			(type default)
+			(width 0.5)
+			(type solid)
 		)
 	)
@@
 		)
 		(stroke
-			(width 0)
-			(type default)
+			(width 0.5)
+			(type solid)
 		)
 	)
@@
 		)
 		(stroke
-			(width 0)
-			(type default)
+			(width 0.5)
+			(type solid)
 		)
 	)
@@
 	(symbol
 		(lib_id "PCM_SparkFun-PowerSymbol:GND")
+		(at 20.32 57.15 0)
+		(unit 1)
+		(body_style 1)
+		(exclude_from_sim no)
+		(in_bom yes)
+		(on_board yes)
+		(in_pos_files yes)
+		(dnp no)
+		(fields_autoplaced yes)
+		(property "Reference" "#PWR013"
+			(at 20.32 63.5 0)
+			(hide yes)
+			(show_name no)
+			(do_not_autoplace no)
+			(effects
+				(font
+					(size 1.27 1.27)
+				)
+			)
+		)
+		(property "Value" "GND"
+			(at 20.32 60.96 0)
+			(show_name no)
+			(do_not_autoplace yes)
+			(effects
+				(font
+					(size 1.27 1.27)
+				)
+			)
+		)
+		(property "Footprint" ""
+			(at 20.32 57.15 0)
+			(hide yes)
+			(show_name no)
+			(do_not_autoplace no)
+			(effects
+				(font
+					(size 1.27 1.27)
+				)
+			)
+		)
+		(property "Datasheet" ""
+			(at 20.32 57.15 0)
+			(hide yes)
+			(show_name no)
+			(do_not_autoplace no)
+			(effects
+				(font
+					(size 1.27 1.27)
+				)
+			)
+		)
+		(property "Description" "Power symbol creates a global label with name \"GND\" , ground"
+			(at 20.32 66.04 0)
+			(hide yes)
+			(show_name no)
+			(do_not_autoplace no)
+			(effects
+				(font
+					(size 1.27 1.27)
+				)
+			)
+		)
+		(pin "1"
+		)
+		(instances
+			(project "Mind_Speak_(Dongle_Board)"
+				(path "/602895f5-aacf-4c92-9095-deb81879ec95"
+					(reference "#PWR013")
+					(unit 1)
+				)
+			)
+		)
+	)
+	(symbol
+		(lib_id "PCM_SparkFun-PowerSymbol:GND")
 		(at 219.71 81.28 0)
 		(unit 1)
@@
 	)
 	(symbol
+		(lib_id "PCM_SparkFun-PowerSymbol:GND")
+		(at 209.55 125.73 0)
+		(unit 1)
+		(body_style 1)
+		(exclude_from_sim no)
+		(in_bom yes)
+		(on_board yes)
+		(in_pos_files yes)
+		(dnp no)
+		(fields_autoplaced yes)
+		(property "Reference" "#PWR014"
+			(at 209.55 132.08 0)
+			(hide yes)
+			(show_name no)
+			(do_not_autoplace no)
+			(effects
+				(font
+					(size 1.27 1.27)
+				)
+			)
+		)
+		(property "Value" "GND"
+			(at 209.55 129.54 0)
+			(show_name no)
+			(do_not_autoplace yes)
+			(effects
+				(font
+					(size 1.27 1.27)
+				)
+			)
+		)
+		(property "Footprint" ""
+			(at 209.55 125.73 0)
+			(hide yes)
+			(show_name no)
+			(do_not_autoplace no)
+			(effects
+				(font
+					(size 1.27 1.27)
+				)
+			)
+		)
+		(property "Datasheet" ""
+			(at 209.55 125.73 0)
+			(hide yes)
+			(show_name no)
+			(do_not_autoplace no)
+			(effects
+				(font
+					(size 1.27 1.27)
+				)
+			)
+		)
+		(property "Description" "Power symbol creates a global label with name \"GND\" , ground"
+			(at 209.55 134.62 0)
+			(hide yes)
+			(show_name no)
+			(do_not_autoplace no)
+			(effects
+				(font
+					(size 1.27 1.27)
+				)
+			)
+		)
+		(pin "1"
+		)
+		(instances
+			(project "Mind_Speak_(Dongle_Board)"
+				(path "/602895f5-aacf-4c92-9095-deb81879ec95"
+					(reference "#PWR014")
+					(unit 1)
+				)
+			)
+		)
+	)
+	(symbol
 		(lib_id "PCM_SparkFun-Resistor:330_0402")
 		(at 261.62 58.42 90)
@@
 		(pin "2"
 		)
+		(pin "4"
+		)
 		(instances

Commit message: Edit in Dongle/Main Boards
Connections:
- net D-: now reaches C3.1, D3.2, J1.2 (D-), R2.1
- net D+: now reaches C2.1, D2.2, J1.3 (D+), R1.1
Changed lines of the file:
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@@
+		)
+	)
+	(label "D+"
+		(at 33.02 43.18 0)
+		(fields_autoplaced yes)
+		(effects
+			(font
+				(size 1.27 1.27)
+			)
+			(justify left bottom)
+		)
+		(property "Net Class" "DP_90R"
+			(at 33.02 44.45 0)
+			(show_name no)
+			(do_not_autoplace no)
+			(effects
+				(font
+					(size 1.27 1.27)
+					(italic yes)
+				)
+				(justify left)
+			)
+		)
+	)
+	(label "D-"
+		(at 33.02 45.72 0)
+		(fields_autoplaced yes)
+		(effects
+			(font
+				(size 1.27 1.27)
+			)
+			(justify left bottom)
+		)
+		(property "Net Class" "DP_90R"
+			(at 33.02 46.99 0)
+			(show_name no)
+			(do_not_autoplace no)
+			(effects
+				(font
+					(size 1.27 1.27)
+					(italic yes)
+				)
+				(justify left)
+			)
 		)
 	)
