File: Hardware_Design/Mind_Speak_(Main_Board)/Mind_Speak_(Main_Board).kicad_sch (KiCad schematic)
At the start: 67 parts, among them J1 microSD, J4 Conn_01x08_Pin, J5 Conn_01x02_Pin, J6 Conn_01x04_Pin, J7 Conn_01x04_Pin, J8 Conn_02x13_Odd_Even, P1 S2B-PH-SM4-TB_LF__SN_, U1 CDBU0130L, U10 PIC32MX250F128B-I_SS, U2 LP5907MFX-3.3, U3 NINA-B30x, U4 TLV70025_SOT23-5, U5 TPS72325DBV, U6 LIS3DH, U7 SN74LVC1G32DCKR, U8 ADS1299, U9 TPS60403DBV

Commit message: Added Dongle Design
Other:
- title: MindSpeak -> MindSpeak_(Main_Board)

Commit message: Edit The main Board
Parts:
- added C3, C41: 18pF, PCM_SparkFun-Capacitor:C_0402_1005Metric, symbol PCM_SparkFun-Capacitor:18pF_0603_50V_5%
- added C40: 10uF, PCM_SparkFun-Capacitor:C_0603_1608Metric, symbol PCM_SparkFun-Capacitor:10uF_0603_10V_20%
- added D7: Blue, PCM_SparkFun-LED:LED_0603_1608Metric_Blue, symbol PCM_SparkFun-LED:LED_Blue_0603
- added R2, R4: 470K, SparkFun-Resistor:R_0402_1005Metric, symbol SparkFun-Resistor:1M_0402
- added R3: 1K, SparkFun-Resistor:R_0402_1005Metric, symbol SparkFun-Resistor:1M_0402
- added SW1, SW2: SW_MEC_5E, Button_Switch_SMD:SW_Push_1P1T_NO_Vertical_Wuerth_434133025816, symbol Switch:SW_MEC_5E
- added Y1: Crystal, PCM_SparkFun-Clock:Crystal-SMD-5x3.2mm, symbol PCM_SparkFun-Clock:Crystal
Connections:
- net VSS is gone; now on net GNDA: U10.19 (VSS), U10.8 (VSS)
- net +2.5VA: now also J8.1 (Pin_1), J8.2 (Pin_2)
- net +3V3: now also J4.1 (Pin_1), J6.3 (Pin_3), U10.13 (VDD), U10.15 (VBUS), U10.23 (VBUS3V3), U10.28 (AVDD), R2.2, SW1.1, SW1.2
- net 1N: now also J8.21 (Pin_21)
- net 1P: now also J8.22 (Pin_22)
- net 2N: now also J8.19 (Pin_19)
- net 2P: now also J8.20 (Pin_20)
- net 3N: now also J8.17 (Pin_17)
- net 3P: now also J8.18 (Pin_18)
- net 4N: now also J8.15 (Pin_15)
- net 4P: now also J8.16 (Pin_16)
- net 5N: now also J8.13 (Pin_13)
- net 5P: now also J8.14 (Pin_14)
- net 6N: now also J8.11 (Pin_11)
- net 6P: now also J8.12 (Pin_12)
- net 7N: now also J8.9 (Pin_9)
- net 7P: now also J8.10 (Pin_10)
- net 8N: now also J8.7 (Pin_7)
- net 8P: now also J8.8 (Pin_8)
- net BIAS: now also J8.5 (Pin_5), J8.6 (Pin_6)
- net BIAS_INV: now also J5.2 (Pin_2)
- net CLK: now also J4.6 (Pin_6)
- net CS1: now also U10.26 (RB15)
- net CS3: now also U10.17 (RB8)
- net CS4: now also U10.16 (RB7)
- net DRDY: now also U10.2 (RA0)
- net GNDA: now also J4.2 (Pin_2), J5.1 (Pin_1), J6.4 (Pin_4), J8.3 (Pin_3), J8.4 (Pin_4), U10.27 (AVSS), C3.1, C40.2, C41.1, R3.1, R4.1, SW2.1, SW2.2
- net INT1: now also U10.14 (RB5)
- net MISO: now also J4.3 (Pin_3), U10.22 (RB11)
- net MOSI: now also J4.7 (Pin_7), U10.3 (RA1)
- net RESET: now also J4.5 (Pin_5), U10.21 (RB10)
- net SCLK: now also J4.4 (Pin_4), U10.25 (RB14)
- net SRB1: now also J8.24 (Pin_24)
- net SRB2: now also J8.23 (Pin_23)
- net VSSA: now also J8.25 (Pin_25), J8.26 (Pin_26)
- net BOOT_EN: now reaches J7.1 (Pin_1)
- net BOOT_EN: now also U10.11 (RB4), R4.2, SW1.3 (K), SW1.4 (A)
- net MCLR: now reaches J7.2 (Pin_2)
- net MCLR: now also U10.1 (MCLR), R2.1, SW2.3 (K), SW2.4 (A)
- net D18: now reaches J7.3 (Pin_3)
- net D18: now also U10.12 (RA4)
- net PGED: now reaches J7.4 (Pin_4)
- net PGED: now also U10.4 (RB0), D7.2 (A)
- net CS2: now reaches J4.8 (Pin_8)
- net CS2: now also U10.18 (RB9)
- net D13: now reaches J6.1 (Pin_1)
- net D13: now also U10.6 (RB2)
- net PGEC: now reaches J6.2 (Pin_2)
- net PGEC: now also U10.5 (RB1)
- net at U10.10 (RA3): now also C41.2, Y1.2
- net at U10.20 (VCAP): now also C40.1
- net RXD: now reaches U10.24 (RB13)
- net TXD: now reaches U10.7 (RB3)
- net at U10.9 (RA2): now also C3.2, Y1.1
- new net: D7.1 (K), R3.2
Other:
- note added: "ADC_CHANNELS"
- note added: "DAISY_BUS"
- note added: "PIC_INTERFACING"
- moved on the sheet: J4, J5, J6, J7, J8, U10

Commit message: Last Edit in main and dongle boards
Parts:
- added J2, J3: Conn_01x05_Pin, Connector_PinHeader_2.54mm:PinHeader_1x05_P2.54mm_Vertical, symbol Connector:Conn_01x05_Pin
- added SW3: SW_MEC_5E, Button_Switch_SMD:SW_Push_1P1T_NO_Vertical_Wuerth_434133025816, symbol Switch:SW_MEC_5E
- added SW4: SPDT_Slide_SMD_6.7x2.6mm, Button_Switch_SMD:SW_SPDT_Shouhan_MSK12C02, symbol PCM_SparkFun-Switch:SPDT_Slide_SMD_6.7x2.6mm
- Y1: value Crystal -> 8MHz
Connections:
- net 3V EN is gone; now on an unnamed net: U2.3 (EN)
- net EGP is gone; now on net EAGP: U3.EGP1 (EGP), U3.EGP10 (EGP), U3.EGP11 (EGP), U3.EGP12 (EGP), U3.EGP2 (EGP), U3.EGP3 (EGP), U3.EGP4 (EGP), U3.EGP5 (EGP), U3.EGP6 (EGP), U3.EGP7 (EGP), U3.EGP8 (EGP), U3.EGP9 (EGP)
- net GND is gone; now on net EAGP: U3.12 (GND), U3.14 (GND), U3.26 (GND), U3.30 (GND), U3.53 (GND), U3.6 (GND)
- net GNDA is gone; now on net EAGP: C1.1, C10.1, C11.2, C12.2, C13.2, C16.2, C17.2, C18.2, C19.2, C2.1, C20.2, C21.2, C22.2, C3.1, C31.1, C32.1, C33.2, C35.2, C36.5, C36.6, C36.7, C36.8, C37.5, C37.6, C37.7, C37.8, C38.5, C38.6, C38.7, C38.8, C39.2, C39.5, C39.6, C39.7, C39.8, C4.5, C4.6, C4.7, C4.8, C40.2, C41.1, C5.1, C6.1, C7.2, C8.1, C9.2, D1.3 (GND), D2.3 (GND), D3.3 (GND), D4.3 (GND), D5.3 (GND), D6.1 (IO1), D6.3 (GND), J1.10 (SHIELD), J1.6 (VSS), J4.2 (Pin_2), J5.1 (Pin_1), J6.4 (Pin_4), J8.3 (Pin_3), J8.4 (Pin_4), P1.2, R3.1, R4.1, RN6.2, RN6.7, SW2.1, SW2.2, U10.19 (VSS), U10.27 (AVSS), U10.8 (VSS), U2.2 (GND), U4.2 (GND), U5.1 (GND), U6.10 (RES), U6.12 (GND), U6.5 (GND), U7.3 (GND), U8.31 (RESV1), U8.33 (DGND), U8.41 (DAISY_IN), U8.49 (DGND), U8.51 (DGND), U8.60 (BIASREF), U8.64 (RESERVED), U9.4 (GND)
- net +3V3: now also SW4.1 (A), SW4.MT1
- net EAGP: now also J2.5 (Pin_5), SW3.1, SW3.2
- net PGEC: now also U3.5 (GPIO_5)
- net RXD: now also U3.2 (GPIO_2)
- net TXD: now also U3.3 (GPIO_3)
- net NINA_PWR: now reaches U3.10 (VCC)
- net NINA_PWR: now also U3.9 (VCC_IO), SW4.2
- net SWD_CLK: now reaches U3.11 (SWDCLK)
- net SWD_CLK: now also J2.2 (Pin_2)
- net SWD_IO: now reaches U3.15 (SWDIO)
- net SWD_IO: now also J2.3 (Pin_3)
- net NINA_RST: now reaches U3.19 (~{RESET})
- net NINA_RST: now also J2.4 (Pin_4), SW3.3 (K), SW3.4 (A)
- net at U3.35 (GPIO_35): now also J3.5 (Pin_5)
- net at U3.36 (GPIO_36): now also J3.4 (Pin_4)
- net at U3.37 (GPIO_37): now also J3.3 (Pin_3)
- net at U3.38 (GPIO_38): now also J3.2 (Pin_2)
- net at U3.39 (GPIO_39): now also J3.1 (Pin_1)
- new net NINA_VCC: J2.1 (Pin_1), SW4.3 (C)
- no-connect marks 20 -> 56
Other:
- note added: "BLE_INTERFACING"
- note added: "GPIO_PINS"
- note added: "NINA_RX"
- note added: "NINA_TX"
- note added: "PIC32_INTERFACING"
- note removed: "PIC_INTERFACING"
- moved on the sheet: J5, J8, U3

Commit message: Edit in Dongle Layout
Parts:
- removed SW4: SPDT_Slide_SMD_6.7x2.6mm, Button_Switch_SMD:SW_SPDT_Shouhan_MSK12C02, symbol PCM_SparkFun-Switch:SPDT_Slide_SMD_6.7x2.6mm
- added S1: SSSS811101, ALPS_Library:SW_SSSS811101, symbol SSSS811101:SSSS811101
- C1, C10, C2, C5, C6, C8: LINK (none) -> https://www2.mouser.com/en/ProductDetail/Murata-Electronics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; VENDOR (none) -> Mouser
- C11, C20, C24, C40, C7: LINK (none) -> https://www.lcsc.com/product-detail/C710916.html?s_z=n_q_GR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; VENDOR (none) -> LCSC
- C12, C15, C17, C19, C26, C28, C29, C31, C32, C33, C34, C35: LINK (none) -> https://www2.mouser.com/en/ProductDetail/YAGEO/CC0402KRX7R5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; VENDOR (none) -> Mouser
- C13, C14, C16, C18, C21, C23, C25, C30: LINK (none) -> https://www2.mouser.com/en/ProductDetail/YAGEO/CC0402KRX7R7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; VENDOR (none) -> Mouser
- C22, C27: LINK (none) -> https://www2.mouser.com/en/ProductDetail/YAGEO/CC1206MKX5R5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; VENDOR (none) -> Mouser
- C3, C41: LINK (none) -> https://www2.mouser.com/en/ProductDetail/YAGEO/CC0402JRNPO9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; VENDOR (none) -> Mouser
- C36, C37, C38, C39, C4: value CKCL44X7R1H102M085AA -> 0.001uF; VENDOR (none) -> **
- C9: value 10nF -> 0.01uF; LINK (none) -> https://www2.mouser.com/en/ProductDetail/YAGEO/CC0402KRX7R7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; VENDOR (none) -> Mouser
- D1, D2, D3, D4, D5, D6, U2, U4, U8: LINK (none) -> https://www2.mouser.com/en/ProductDetail/Texas-Instruments/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; VENDOR (none) -> Mouser
- D7: LINK (none) -> https://www2.mouser.com/en/ProductDetail/LITEON/LTST-C193TB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; VENDOR (none) -> Mouser
- J1: footprint PCM_SparkFun-Connector:microSD_External_Pin -> SparkFun-Connector:CUI_MSD-1-A; LINK (none) -> https://www2.mouser.com/en/ProductDetail/Same-Sky/MSD-1-A?q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; VENDOR (none) -> Mouser
- J2, J3, J4, J5, J6, J7: LINK (none) -> https://microohm-eg.com/pin-header-2-54mm-1x40-pin-male-sin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; VENDOR (none) -> MicroOhm
- J8: LINK (none) -> https://microohm-eg.com/2-54mm-0-100-pin-header-male-2x40-r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; VENDOR (none) -> MicroOhm
- P1: footprint S2B-PH-SM4-TB_LF__SN_:JST_S2B-PH-SM4-TB_LF__SN_ -> JST_Library:JST_S2B-PH-SM4-TB_LF__SN_; LINK (none) -> https://www.lcsc.com/product-detail/C295747.html; VENDOR (none) -> LCSC
- R1: LINK (none) -> https://www2.mouser.com/en/ProductDetail/YAGEO/RC0402JR-071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; VENDOR (none) -> Mouser
- R2, R4: LINK (none) -> https://www2.mouser.com/en/ProductDetail/YAGEO/RC0402JR-074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; VENDOR (none) -> Mouser
- R3: LINK (none) -> https://www2.mouser.com/en/ProductDetail/YAGEO/RT0402FRE071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; VENDOR (none) -> Mouser
- RN2, RN3, RN4, RN5, RN6: LINK (none) -> https://www2.mouser.com/en/ProductDetail/Bourns/CAY16-2201F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; VENDOR (none) -> Mouser
- SW1, SW2, SW3: LINK (none) -> https://www2.mouser.com/en/ProductDetail/CK/PTS810SJK250SMT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; VENDOR (none) -> Mouser
- U1: footprint (none) -> Comchip_Library:CDBU; LINK (none) -> https://www2.mouser.com/en/ProductDetail/Comchip-Technology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; VENDOR (none) -> Mouser
- U10: LINK (none) -> https://www2.mouser.com/en/ProductDetail/Microchip-Technolo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; VENDOR (none) -> Mouser
- U3: LINK (none) -> https://www2.mouser.com/en/ProductDetail/u-blox/NINA-B306-0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; VENDOR (none) -> Mouser
- U5: value TPS72325DBV -> TPS72325DBVR; LINK (none) -> https://www.lcsc.com/product-detail/C69932.html?s_z=n_q_TPS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; VENDOR (none) -> Mouser
- U6: LINK (none) -> https://www2.mouser.com/en/ProductDetail/STMicroelectronics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; VENDOR (none) -> Mouser
- U7: footprint SN74LVC1G32DCKR:SOT65P210X110-5N -> TI_Library:SOT65P210X110-5N; LINK (none) -> https://www2.mouser.com/en/ProductDetail/Texas-Instruments/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; VENDOR (none) -> Mouser
- U9: LINK (none) -> https://www.lcsc.com/product-detail/C11338.html?s_z=n_q_TPS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; VENDOR (none) -> LCSC
- Y1: footprint PCM_SparkFun-Clock:Crystal-SMD-5x3.2mm -> Abracon_Library:XTAL_ABMM2-8.000MHZ-E2-T; LINK (none) -> https://www2.mouser.com/en/ProductDetail/ABRACON/ABMM2-8.00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; VENDOR (none) -> Mouser
Connections:
- net +3V3: now also S1.1
- net NINA_PWR: now also S1.2
- net NINA_VCC: now also S1.3
Other:
- moved on the sheet: J3, SW3, U3

Commit message: Edit In Layout Of Main Board
Parts:
- removed J3: Conn_01x05_Pin, Connector_PinHeader_2.54mm:PinHeader_1x05_P2.54mm_Vertical, symbol Connector:Conn_01x05_Pin
- removed Y1: 8MHz, Abracon_Library:XTAL_ABMM2-8.000MHZ-E2-T, symbol PCM_SparkFun-Clock:Crystal
- added C41: 0.1uF, PCM_SparkFun-Capacitor:C_0402_1005Metric, symbol PCM_SparkFun-Capacitor:0.1uF_0402_16V_10%
- added C42: 10uF, PCM_SparkFun-Capacitor:C_0603_1608Metric, symbol PCM_SparkFun-Capacitor:10uF_0603_10V_20%
- added H1, H2, H3, H4: MountingHole_Pad, MountingHole:MountingHole_3.2mm_M3_Pad, symbol Mechanical:MountingHole_Pad
- added J8: Conn_01x05_Pin, Connector_PinHeader_2.54mm:PinHeader_1x05_P2.54mm_Vertical, symbol Connector:Conn_01x05_Pin
- added Y1: ABMM2-8.000MHZ-E2-T, Abracon_Library:XTAL_ABMM2-8.000MHZ-E2-T, symbol ABMM2-8.000MHZ-E2-T:ABMM2-8.000MHZ-E2-T
- C12: renamed from C8; LINK https://www2.mouser.com/en/ProductDetail/Murata-Electronics/GRM155C80J225ME95D?qs=eeBpzGFlv%252B%2FrWGjWqjxzrQ%3D%3D&srsltid=AfmBOooN7zLjP1ysYE6i-5gamX0EZDBjMpP8ik1ZROxz0EmXyiMfHLCA -> https://www2.mouser.com/en/ProductDetail/Murata-Electronics/GRM155R61C225KE44D?qs=K0Sa7bCb58LeAAXFhnh74A%3D%3D&srsltid=AfmBOoo586f-fBnXaQR3ZmOT4GDLYhDBoqTxzex_jrWoladTqBGt2nID
- C15: renamed from C5; LINK https://www2.mouser.com/en/ProductDetail/Murata-Electronics/GRM155C80J225ME95D?qs=eeBpzGFlv%252B%2FrWGjWqjxzrQ%3D%3D&srsltid=AfmBOooN7zLjP1ysYE6i-5gamX0EZDBjMpP8ik1ZROxz0EmXyiMfHLCA -> https://www2.mouser.com/en/ProductDetail/Murata-Electronics/GRM155R61C225KE44D?qs=K0Sa7bCb58LeAAXFhnh74A%3D%3D&srsltid=AfmBOoo586f-fBnXaQR3ZmOT4GDLYhDBoqTxzex_jrWoladTqBGt2nID
- C22: renamed from C36; LINK (none) -> https://eu.mouser.com/en/ProductDetail/TDK/CKCL44X7R1H102M0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; VENDOR ** -> **Mouser
- C25: renamed from C10; LINK https://www2.mouser.com/en/ProductDetail/Murata-Electronics/GRM155C80J225ME95D?qs=eeBpzGFlv%252B%2FrWGjWqjxzrQ%3D%3D&srsltid=AfmBOooN7zLjP1ysYE6i-5gamX0EZDBjMpP8ik1ZROxz0EmXyiMfHLCA -> https://www2.mouser.com/en/ProductDetail/Murata-Electronics/GRM155R61C225KE44D?qs=K0Sa7bCb58LeAAXFhnh74A%3D%3D&srsltid=AfmBOoo586f-fBnXaQR3ZmOT4GDLYhDBoqTxzex_jrWoladTqBGt2nID
- C27: renamed from C6; LINK https://www2.mouser.com/en/ProductDetail/Murata-Electronics/GRM155C80J225ME95D?qs=eeBpzGFlv%252B%2FrWGjWqjxzrQ%3D%3D&srsltid=AfmBOooN7zLjP1ysYE6i-5gamX0EZDBjMpP8ik1ZROxz0EmXyiMfHLCA -> https://www2.mouser.com/en/ProductDetail/Murata-Electronics/GRM155R61C225KE44D?qs=K0Sa7bCb58LeAAXFhnh74A%3D%3D&srsltid=AfmBOoo586f-fBnXaQR3ZmOT4GDLYhDBoqTxzex_jrWoladTqBGt2nID
- C28: renamed from C37; LINK (none) -> https://eu.mouser.com/en/ProductDetail/TDK/CKCL44X7R1H102M0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; VENDOR ** -> **Mouser
- C36: renamed from C38; LINK (none) -> https://eu.mouser.com/en/ProductDetail/TDK/CKCL44X7R1H102M0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; VENDOR ** -> **Mouser
- C38: renamed from C39; LINK (none) -> https://eu.mouser.com/en/ProductDetail/TDK/CKCL44X7R1H102M0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; VENDOR ** -> **Mouser
- C8: renamed from C4; LINK (none) -> https://eu.mouser.com/en/ProductDetail/TDK/CKCL44X7R1H102M0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; VENDOR ** -> **Mouser
- C9: renamed from C2; LINK https://www2.mouser.com/en/ProductDetail/Murata-Electronics/GRM155C80J225ME95D?qs=eeBpzGFlv%252B%2FrWGjWqjxzrQ%3D%3D&srsltid=AfmBOooN7zLjP1ysYE6i-5gamX0EZDBjMpP8ik1ZROxz0EmXyiMfHLCA -> https://www2.mouser.com/en/ProductDetail/Murata-Electronics/GRM155R61C225KE44D?qs=K0Sa7bCb58LeAAXFhnh74A%3D%3D&srsltid=AfmBOoo586f-fBnXaQR3ZmOT4GDLYhDBoqTxzex_jrWoladTqBGt2nID
- renumbered C20 to C1, C13 to C10, C16 to C11, C12 to C13, C17 to C14, C27 to C16, C14 to C17, C26 to C19, C21 to C2, C15 to C20, C19 to C21, C9 to C23, C29 to C24, C30 to C26, C11 to C29, C33 to C3, C28 to C30, C7 to C31, C25 to C32, C24 to C33, C31 to C34, C32 to C35, C23 to C37, C3 to C39, C22 to C4, C41 to C40, C40 to C43, C1 to C5, C34 to C6, C35 to C7, D6 to D4, D4 to D5, D5 to D6, J6 to J2, J8 to J3, J7 to J4, J4 to J5, J5 to J6, J2 to J7, R3 to R2, R4 to R3, R2 to R4, RN2 to RN1, RN3 to RN2, RN4 to RN3, RN5 to RN4, RN6 to RN5, SW3 to SW1, SW1 to SW3, U7 to U1, U9 to U2, U1 to U3, U6 to U4, U2 to U5, U5 to U6, U4 to U7, U3 to U9
Connections:
- net +2.5VA: now also J3.25 (Pin_25), J3.26 (Pin_26); no longer J3.1 (Pin_1), J3.2 (Pin_2)
- net 1N: now also J3.5 (Pin_5); no longer J3.21 (Pin_21)
- net 1P: now also J3.6 (Pin_6); no longer J3.22 (Pin_22)
- net 2N: now also J3.7 (Pin_7); no longer J3.19 (Pin_19)
- net 2P: now also J3.8 (Pin_8); no longer J3.20 (Pin_20)
- net 3N: now also J3.9 (Pin_9); no longer J3.17 (Pin_17)
- net 3P: now also J3.10 (Pin_10); no longer J3.18 (Pin_18)
- net 4N: now also J3.11 (Pin_11); no longer J3.15 (Pin_15)
- net 4P: now also J3.12 (Pin_12); no longer J3.16 (Pin_16)
- net 6N: now also J3.15 (Pin_15); no longer J3.11 (Pin_11)
- net 6P: now also J3.16 (Pin_16); no longer J3.12 (Pin_12)
- net 7N: now also J3.17 (Pin_17); no longer J3.9 (Pin_9)
- net 7P: now also J3.18 (Pin_18); no longer J3.10 (Pin_10)
- net 8N: now also J3.19 (Pin_19); no longer J3.7 (Pin_7)
- net 8P: now also J3.20 (Pin_20); no longer J3.8 (Pin_8)
- net BIAS: now also J3.21 (Pin_21), J3.22 (Pin_22); no longer J3.5 (Pin_5), J3.6 (Pin_6)
- net EAGP: now also J3.23 (Pin_23), J3.24 (Pin_24), S1.4 (SHIELD), C41.2, C42.2, H1.1, H2.1, H3.1, H4.1, Y1.2 (GND), Y1.4 (GND); no longer J3.3 (Pin_3), J3.4 (Pin_4)
- net NINA_PWR: now also C41.1, C42.1
- net SRB1: now also J3.4 (Pin_4); no longer J3.24 (Pin_24)
- net SRB2: now also J3.3 (Pin_3); no longer J3.23 (Pin_23)
- net VSSA: now also J3.1 (Pin_1), J3.2 (Pin_2); no longer J3.25 (Pin_25), J3.26 (Pin_26)
- net at C40.2, U10.10 (RA3): now also Y1.3
- net at C39.2, U10.9 (RA2): now also Y1.1
- net at U9.18 (GPIO_18): now also J8.5 (Pin_5)
- net at U9.20 (GPIO_20): now also J8.4 (Pin_4)
- net at U9.21 (GPIO_21): now also J8.3 (Pin_3)
- net at U9.22 (GPIO_22): now also J8.2 (Pin_2)
- net at U9.23 (GPIO_23): now also J8.1 (Pin_1)
- net -V renamed -3V3
- no-connect marks 56 -> 58
Other:
- moved on the sheet: C15, C27, C31, C39, C40, C43, D7, J5, R2, R3, R4, SW1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

Commit message: Edit in Dongle/Main Boards
Parts:
- H1, H2, H3, H4: now in the parts list
Changed lines of the file:
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@@
 		(body_style 1)
 		(exclude_from_sim no)
-		(in_bom no)
+		(in_bom yes)
 		(on_board yes)
 		(in_pos_files yes)
@@
 		(body_style 1)
 		(exclude_from_sim no)
-		(in_bom no)
+		(in_bom yes)
 		(on_board yes)
 		(in_pos_files yes)
@@
 		(body_style 1)
 		(exclude_from_sim no)
-		(in_bom no)
+		(in_bom yes)
 		(on_board yes)
 		(in_pos_files yes)
@@
 		(body_style 1)
 		(exclude_from_sim no)
-		(in_bom no)
+		(in_bom yes)
 		(on_board yes)
 		(in_pos_files yes)

Commit message: Last Update and Updated the BOM List
Parts:
- H1, H2, H3, H4: now left out of the parts list
Changed lines of the file:
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@@
 		(body_style 1)
 		(exclude_from_sim no)
-		(in_bom yes)
-		(on_board yes)
+		(in_bom no)
+		(on_board no)
 		(in_pos_files yes)
 		(dnp no)
@@
 		(body_style 1)
 		(exclude_from_sim no)
-		(in_bom yes)
-		(on_board yes)
+		(in_bom no)
+		(on_board no)
 		(in_pos_files yes)
 		(dnp no)
@@
 		(body_style 1)
 		(exclude_from_sim no)
-		(in_bom yes)
-		(on_board yes)
+		(in_bom no)
+		(on_board no)
 		(in_pos_files yes)
 		(dnp no)
@@
 		(body_style 1)
 		(exclude_from_sim no)
-		(in_bom yes)
-		(on_board yes)
+		(in_bom no)
+		(on_board no)
 		(in_pos_files yes)
 		(dnp no)
